Commit message: fixed urdf axes

File: urdf/robot.urdf (robot description, URDF)
Before this commit: robot edwin, 6 links, 5 joints
Joints:
- joint joint_2: axis 0 0 -1 -> 0 0 1
- joint joint_4: axis 0 0 1 -> 0 0 -1

Commit message: renamed joints

File: urdf/robot.urdf (robot description, URDF)
Before this commit: robot edwin, 6 links, 5 joints
Joints:
- removed joint joint_1
- removed joint joint_2
- removed joint joint_3
- removed joint joint_4
- removed joint joint_5
- added joint elbow: type continuous, parent link_2, child link_3, origin xyz=-0.375 0 0 rpy=0 0 -1.1442E-17, axis 0 0 1
- added joint hand: type continuous, parent link_3, child link_4, origin xyz=-0.375 0 0 rpy=3.1416 0 3.1416, axis 0 0 -1
- added joint shoulder: type continuous, parent link_1, child link_2, origin xyz=0 0 0.32173 rpy=1.5708 1.5708 3.1416, axis 0 0 1
- added joint waist: type continuous, parent base_link, child link_1, origin xyz=0 0 0.0332679193608537 rpy=-6.12303176911189E-17 0 0, axis 0 0 -1
- added joint wrist: type continuous, parent link_4, child link_5, origin xyz=0.042405 0 -0.0244 rpy=0 -1.5708 0, axis 0 0 -1
